File: Electrical_schematics/Electrical_schematics_V2/Electrical_schematics_V2.kicad_sch (KiCad schematic)
At the start: 8 parts, among them SW2 SW_Push, U1 VL53L4CXV0DH_1, U6 XIAO ESP32C3

Commit message: file changes to PCB version history
Connections:
- net 3.3V: now also R3.2
- net VCC: no longer R3.2
Changed lines of the file:
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@@
 	)
 	(symbol
-		(lib_id "Adafruit VL53L4CX-eagle-import:VCC")
+		(lib_id "Adafruit VL53L4CX-eagle-import:2.8V")
 		(at 173.99 193.04 0)
 		(unit 1)
@@
 		(on_board yes)
 		(dnp no)
-		(property "Reference" "#P+03"
+		(property "Reference" "#U$01"
 			(at 173.99 193.04 0)
 			(effects
@@
 			)
 		)
-		(property "Value" "VCC"
-			(at 171.45 195.58 90)
+		(property "Value" "3.3V"
+			(at 172.466 192.024 0)
 			(effects
 				(font
-					(size 1.778 1.5113)
+					(size 1.27 1.0795)
 				)
 				(justify left bottom)
@@
 		)
 		(instances
-			(project "Electrical_schematics"
+			(project "Electrical_schematics_V2"
 				(path "/3dd2c12c-1a32-422a-803d-8f2ed5a6c585"
-					(reference "#P+03")
+					(reference "#U$01")
 					(unit 1)
 				)
